File: Wifi_Shielf_KiCad_Files/_saved_OpenBCI_Wifi_Shield.sch (KiCad schematic (older format))
At the start: 22 parts, among them P1 CONN_01X04, P10 CONN_01X04, P2 CONN_01X02, P4 CONN_01X02, P5 CONN_01X02, P6 CONN_01X02, P7 CONN_01X08, P8 CONN_01X08, P9 CONN_01X04, SW1 TACT_SWITCH, SW2 TACT_SWITCH, U1 ESP-12E, U2 AP2112

Commit message: Brought in board template
Parts:
- U1: footprint OpenBCI:SSSS810701 SSSS810701 -> ESP8266:ESP-12E
Changed lines of the file:
@@
 F 0 "U1" H 4350 2000 50  0000 C CNN
 F 1 "ESP-12E" H 4350 2200 50  0000 C CNN
-F 2 "OpenBCI:SSSS810701SSSS810701" H 4350 2100 50  0001 C CNN
+F 2 "ESP8266:ESP-12E" H 4350 2100 50  0001 C CNN
 F 3 "" H 4350 2100 50  0001 C CNN
 	1    4350 2100

Commit message: saving
Parts:
- P1, P10, P9: footprint Pin_Headers:Pin_Header_Straight_1x04_Pitch2.54mm -> Socket_Strips:Socket_Strip_Straight_1x04
- P4, P5, P6: footprint Pin_Headers:Pin_Header_Straight_1x02_Pitch2.54mm -> Socket_Strips:Socket_Strip_Straight_1x02
- P7, P8: footprint OpenBCI:Pin_Header_Straight_1x08 -> Socket_Strips:Socket_Strip_Straight_1x08
- SW1, SW2: footprint OpenBCI:SSSS810701 SSSS810701 -> OpenBCI:PTS810
Changed lines of the file:
@@
 F 0 "P8" H 10050 4650 50  0000 C CNN
 F 1 "CONN_01X08" V 10150 4200 50  0000 C CNN
-F 2 "OpenBCI:Pin_Header_Straight_1x08" H 10050 4200 50  0001 C CNN
+F 2 "Socket_Strips:Socket_Strip_Straight_1x08" H 10050 4200 50  0001 C CNN
 F 3 "" H 10050 4200 50  0000 C CNN
 	1    10050 4200
@@
 F 0 "P7" H 10050 3550 50  0000 C CNN
 F 1 "CONN_01X08" V 10150 3100 50  0000 C CNN
-F 2 "OpenBCI:Pin_Header_Straight_1x08" H 10050 3100 50  0001 C CNN
+F 2 "Socket_Strips:Socket_Strip_Straight_1x08" H 10050 3100 50  0001 C CNN
 F 3 "" H 10050 3100 50  0000 C CNN
 	1    10050 3100
@@
 F 0 "P9" H 10050 5350 50  0000 C CNN
 F 1 "CONN_01X04" V 10150 5100 50  0000 C CNN
-F 2 "Pin_Headers:Pin_Header_Straight_1x04_Pitch2.54mm" H 10050 5100 50  0001 C CNN
+F 2 "Socket_Strips:Socket_Strip_Straight_1x04" H 10050 5100 50  0001 C CNN
 F 3 "" H 10050 5100 50  0000 C CNN
 	1    10050 5100
@@
 F 0 "P10" H 10050 6050 50  0000 C CNN
 F 1 "CONN_01X04" V 10150 5800 50  0000 C CNN
-F 2 "Pin_Headers:Pin_Header_Straight_1x04_Pitch2.54mm" H 10050 5800 50  0001 C CNN
+F 2 "Socket_Strips:Socket_Strip_Straight_1x04" H 10050 5800 50  0001 C CNN
 F 3 "" H 10050 5800 50  0000 C CNN
 	1    10050 5800
@@
 F 0 "P6" H 10050 2300 50  0000 C CNN
 F 1 "CONN_01X02" V 10150 2150 50  0000 C CNN
-F 2 "Pin_Headers:Pin_Header_Straight_1x02_Pitch2.54mm" H 10050 2150 50  0001 C CNN
+F 2 "Socket_Strips:Socket_Strip_Straight_1x02" H 10050 2150 50  0001 C CNN
 F 3 "" H 10050 2150 50  0000 C CNN
 	1    10050 2150
@@
 F 0 "P5" H 10050 1700 50  0000 C CNN
 F 1 "CONN_01X02" V 10150 1550 50  0000 C CNN
-F 2 "Pin_Headers:Pin_Header_Straight_1x02_Pitch2.54mm" H 10050 1550 50  0001 C CNN
+F 2 "Socket_Strips:Socket_Strip_Straight_1x02" H 10050 1550 50  0001 C CNN
 F 3 "" H 10050 1550 50  0000 C CNN
 	1    10050 1550
@@
 F 0 "P4" H 10050 1150 50  0000 C CNN
 F 1 "CONN_01X02" V 10150 1000 50  0000 C CNN
-F 2 "Pin_Headers:Pin_Header_Straight_1x02_Pitch2.54mm" H 10050 1000 50  0001 C CNN
+F 2 "Socket_Strips:Socket_Strip_Straight_1x02" H 10050 1000 50  0001 C CNN
 F 3 "" H 10050 1000 50  0000 C CNN
 	1    10050 1000
@@
 F 0 "P1" H 3800 5100 50  0000 C CNN
 F 1 "CONN_01X04" V 3900 4850 50  0000 C CNN
-F 2 "Pin_Headers:Pin_Header_Straight_1x04_Pitch2.54mm" H 3800 4850 50  0001 C CNN
+F 2 "Socket_Strips:Socket_Strip_Straight_1x04" H 3800 4850 50  0001 C CNN
 F 3 "" H 3800 4850 50  0000 C CNN
 	1    3800 4850
@@
 F 0 "SW2" H 7300 2310 50  0000 C CNN
 F 1 "TACT_SWITCH" H 7150 2000 50  0000 C CNN
-F 2 "OpenBCI:SSSS810701SSSS810701" H 7150 2200 50  0001 C CNN
+F 2 "OpenBCI:PTS810" H 7150 2200 50  0001 C CNN
 F 3 "" H 7150 2200 50  0000 C CNN
 	1    7150 2200
@@
 F 0 "SW1" H 2650 1910 50  0000 C CNN
 F 1 "TACT_SWITCH" H 2500 1600 50  0000 C CNN
-F 2 "OpenBCI:SSSS810701SSSS810701" H 2500 1800 50  0001 C CNN
+F 2 "OpenBCI:PTS810" H 2500 1800 50  0001 C CNN
 F 3 "" H 2500 1800 50  0000 C CNN
 	1    2500 1800

Commit message: saving
Parts:
- U1: footprint ESP8266:ESP-12E -> OpenBCI_Wifi_Shield:ESP-12E-SMD
Connections:
- net +BATT: now also P2.1 (P1); no longer P2.2 (P2)
- net GND: now also P2.2 (P2); no longer P2.1 (P1)
Changed lines of the file:
@@
 F 3 "" H 5150 5000 50  0000 C CNN
 	1    5150 5000
-	-1   0    0    1
+	-1   0    0    -1
 $EndComp
 $Comp
@@
 F 0 "U1" H 4350 2000 50  0000 C CNN
 F 1 "ESP-12E" H 4350 2200 50  0000 C CNN
-F 2 "ESP8266:ESP-12E" H 4350 2100 50  0001 C CNN
+F 2 "OpenBCI_Wifi_Shield:ESP-12E-SMD" H 4350 2100 50  0001 C CNN
 F 3 "" H 4350 2100 50  0001 C CNN
 	1    4350 2100

Commit message: Finish routing
Parts:
- removed P2: CONN_01X02, OpenBCI:JST_RA_SMT, symbol CONN_01X02
- added P2: CONN_01X04, OpenBCI:JST_RA_SMT, symbol CONN_01X04
Connections:
- net +BATT: now also P2.1 (P1), P2.3 (P3)
- net GND: now also P2.2 (P2), P2.4 (P4)
Changed lines of the file:
@@
-$EndComp
-$Comp
-L CONN_01X02 P2
-U 1 1 58826B47
-P 5150 5000
-F 0 "P2" H 5150 5150 50  0000 C CNN
-F 1 "CONN_01X02" V 5250 5000 50  0000 C CNN
-F 2 "OpenBCI:JST_RA_SMT" H 5150 5000 50  0001 C CNN
-F 3 "" H 5150 5000 50  0000 C CNN
-	1    5150 5000
-	-1   0    0    -1
 $EndComp
 $Comp
@@
 L +BATT #PWR08
 U 1 1 5886A193
-P 5500 4850
-F 0 "#PWR08" H 5500 4700 50  0001 C CNN
-F 1 "+BATT" H 5500 4990 50  0000 C CNN
-F 2 "" H 5500 4850 50  0000 C CNN
-F 3 "" H 5500 4850 50  0000 C CNN
-	1    5500 4850
+P 5450 4750
+F 0 "#PWR08" H 5450 4600 50  0001 C CNN
+F 1 "+BATT" H 5450 4890 50  0000 C CNN
+F 2 "" H 5450 4750 50  0000 C CNN
+F 3 "" H 5450 4750 50  0000 C CNN
+	1    5450 4750
 	1    0    0    -1
 $EndComp
@@
 L GND #PWR09
 U 1 1 5886A1D4
-P 5500 5200
-F 0 "#PWR09" H 5500 4950 50  0001 C CNN
-F 1 "GND" H 5500 5050 50  0000 C CNN
-F 2 "" H 5500 5200 50  0000 C CNN
-F 3 "" H 5500 5200 50  0000 C CNN
-	1    5500 5200
+P 5700 5050
+F 0 "#PWR09" H 5700 4800 50  0001 C CNN
+F 1 "GND" H 5700 4900 50  0000 C CNN
+F 2 "" H 5700 5050 50  0000 C CNN
+F 3 "" H 5700 5050 50  0000 C CNN
+	1    5700 5050
 	1    0    0    -1
 $EndComp
@@
 	7900 5950 7900 3850
 Wire Wire Line
-	5500 4950 5500 4850
-Wire Wire Line
-	5350 4950 5500 4950
-Wire Wire Line
-	5500 5050 5500 5200
-Wire Wire Line
-	5350 5050 5500 5050
+	5700 4950 5700 5050
+Wire Wire Line
+	5250 4950 5700 4950
 Wire Wire Line
 	5850 5550 6700 5550
@@
 	2150 1900 2150 1800
 Connection ~ 2150 1800
+$Comp
+L CONN_01X04 P2
+U 1 1 5887F7D9
+P 5050 5000
+F 0 "P2" H 5050 5250 50  0000 C CNN
+F 1 "CONN_01X04" V 5150 5000 50  0000 C CNN
+F 2 "OpenBCI:JST_RA_SMT" H 5050 5000 50  0001 C CNN
+F 3 "" H 5050 5000 50  0000 C CNN
+	1    5050 5000
+	-1   0    0    -1
+$EndComp
+Wire Wire Line
+	5450 4750 5450 4850
+Wire Wire Line
+	5450 4850 5250 4850
+Wire Wire Line
+	5250 5050 5350 5050
+Wire Wire Line
+	5350 5050 5350 4850
+Connection ~ 5350 4850
+Wire Wire Line
+	5250 5150 5550 5150
+Wire Wire Line
+	5550 5150 5550 4950
+Connection ~ 5550 4950
 $EndSCHEMATC
