File: Wifi_Shielf_KiCad_Files/HARDWARE_FILTERS.sch (KiCad schematic (older format))
At the start: 15 parts, among them U4 TPD4E1B06, U5 TPD4E1B06, U6 TPD4E1B06, U7 TPD4E1B06, U8 TPD4E1B06

Commit message: ADD: ADS
Connections:
- net SRB1: no longer R13.3, U8.1 (IO1)
- net SRB2: no longer R13.7, U8.4 (IO3)
- new net: R13.3, U8.1 (IO1)
- new net: R13.7, U8.4 (IO3)
Changed lines of the file:
@@
 $EndComp
 Connection ~ 5050 6900
-Text GLabel 2000 5650 0    60   Input ~ 0
+Text GLabel 1900 4600 0    60   Input ~ 0
 SRB1
 Wire Wire Line
@@
 Connection ~ 8350 5150
 Connection ~ 8400 5050
-Text GLabel 2000 6050 0    60   Input ~ 0
+Text GLabel 1850 5000 0    60   Input ~ 0
 SRB2
 Text GLabel 5350 5850 2    60   Input ~ 0
